File: hardware/adapter.kicad_sch (KiCad schematic)
At the start: 2 parts

Commit message: hardware: updated board design (reference renumbering, LED polarity fix, crystal symbol upgrade)
Replaces the schematics/PCB/project file with the latest design. Key
changes, verified before committing (netlist-check.py: 124 checks, 0
failures; ERC unchanged at 3 known pin_not_driven findings on W5500 SPI
inputs, same severity-policy artifact as before):

- Component reference designators changed from descriptive names
  (R_ATN, C_3V3, D_BR1, etc.) to plain auto-numbered ones (R15, C9, D1,
  etc.) -- intentional, since descriptive names were ending up on the
  silkscreen; they belong in the BOM instead. docs/netlist-spec.nets
  updated to match via a UUID-verified old-ref -> new-ref mapping (every
  renamed symbol's KiCad UUID was unchanged, confirming these are pure
  renames with no electrical difference), not a hand transcription.
- LED1's wiring was corrected: the old schematic had its anode tied to
  GND and cathode driven by LED_A (backwards -- confirmed via each net's
  pinfunction annotation in the exported netlist, K_1/A_2, which is
  fixed by the Device:LED symbol regardless of reference numbering).
  The new schematic has cathode-to-GND, anode-to-LED_A, the correct
  orientation.
- X1/X2 changed from Device:Crystal (2-pin) to Device:Crystal_GND24
  (4-pin, case-ground on pins 2/4) -- a more accurate symbol for the
  real SMD crystal package. netlist-spec.nets updated accordingly
  (XOUT/ETH_XO now reference pin 3, GND gained the four case pins).

mcu.kicad_sch was supplied separately (missing from the first archive);
confirmed it has no further sub-sheet references and all its symbols'
footprint names resolve against the existing hardware/lib/adapter.pretty/
library, which was deliberately left untouched along with fp-lib-table,
sym-lib-table, and .konnect/ -- none of those changed in this update.
Parts:
- removed H1, H2: MountingHole_Pad, MountingHole:MountingHole_3.2mm_M3_Pad, symbol Mechanical:MountingHole_Pad
