File: hardware/power_gate.kicad_sch (KiCad schematic)
At the start: 15 parts, among them J4 PWR_SEL, Q1 AO3401A, Q2 2N7002, U5 AP2114H-3.3TRG1, U6 TPS3839G33DBZR

Commit message: hardware: updated board design (reference renumbering, LED polarity fix, crystal symbol upgrade)
Replaces the schematics/PCB/project file with the latest design. Key
changes, verified before committing (netlist-check.py: 124 checks, 0
failures; ERC unchanged at 3 known pin_not_driven findings on W5500 SPI
inputs, same severity-policy artifact as before):

- Component reference designators changed from descriptive names
  (R_ATN, C_3V3, D_BR1, etc.) to plain auto-numbered ones (R15, C9, D1,
  etc.) -- intentional, since descriptive names were ending up on the
  silkscreen; they belong in the BOM instead. docs/netlist-spec.nets
  updated to match via a UUID-verified old-ref -> new-ref mapping (every
  renamed symbol's KiCad UUID was unchanged, confirming these are pure
  renames with no electrical difference), not a hand transcription.
- LED1's wiring was corrected: the old schematic had its anode tied to
  GND and cathode driven by LED_A (backwards -- confirmed via each net's
  pinfunction annotation in the exported netlist, K_1/A_2, which is
  fixed by the Device:LED symbol regardless of reference numbering).
  The new schematic has cathode-to-GND, anode-to-LED_A, the correct
  orientation.
- X1/X2 changed from Device:Crystal (2-pin) to Device:Crystal_GND24
  (4-pin, case-ground on pins 2/4) -- a more accurate symbol for the
  real SMD crystal package. netlist-spec.nets updated accordingly
  (XOUT/ETH_XO now reference pin 3, GND gained the four case pins).

mcu.kicad_sch was supplied separately (missing from the first archive);
confirmed it has no further sub-sheet references and all its symbols'
footprint names resolve against the existing hardware/lib/adapter.pretty/
library, which was deliberately left untouched along with fp-lib-table,
sym-lib-table, and .konnect/ -- none of those changed in this update.
Parts:
- C23: renamed from C_3V3; LCSC (none) -> C28323
- Q1: LCSC (none) -> C15127
- Q2: LCSC (none) -> C8545
- U5: LCSC (none) -> C150716
- U6: LCSC (none) -> C485802
- renumbered C_LDOin1 to C16, C_BULK1 to C20, C_LDOout1 to C24, C_G1 to C4, R_G2 to R6, R_G1 to R8
Other:
- note added: "FAIL-SAFE: with +3V3 absent U6 is unpowered, R6 holds Q2 off and R8 holds Q1's gate at its source, so +5V_XCVR is dead."
- note added: "TIMING: U6 holds RESET asserted ~200 ms after the rail is good; R8 * C4 then ramp Q1 on (inrush limit, R-HW-051)."
- note removed: "FAIL-SAFE: with +3V3 absent U6 is unpowered, R_G2 holds Q2 off and R_G1 holds Q1's gate at its source, so +5V_XCVR is dead."
- note removed: "TIMING: U6 holds RESET asserted ~200 ms after the rail is good; R_G1 * C_G then ramp Q1 on (inrush limit, R-HW-051)."
